File: esd_sensor.kicad_sch (KiCad schematic)
At the start: 11 parts, among them J2 conn2x1_100mil, Q1 MMBF4117, U1 TLV9151

Commit message: U1 mfg partnumber updated
Parts:
- U1: MFG PN TLV9151SIDBVR -> TLV9151IDBVR
Changed lines of the file:
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@@
 			)
 		)
-		(property "MFG PN" "TLV9151SIDBVR"
+		(property "MFG PN" "TLV9151IDBVR"
 			(at 101.346 58.166 0)
 			(effects
